File: Hardware/Swamper.kicad_pcb (KiCad board)
At the start: 2 copper layers, 39.3 x 63.7 mm, 10 parts, among them J1 MPU6050, J2 Sensor de temperatura, J3 Entrada, J4 Entrada, U1 ESP32, U2 SEN-12650, U3 Mini360

Commit message: Actualizacion de repositorio
Parts:
- removed U3: Mini360, MixLib:Mini360_step-down
- added C1: C, Capacitor_SMD:C_Elec_5x5.8, F.Cu at (155.3, 73.6)
- added C2: C, Capacitor_SMD:C_0805_2012Metric_Pad1.18x1.45mm_HandSolder, F.Cu at (132.3, 73.8)
- added C3: C, Capacitor_SMD:C_0805_2012Metric_Pad1.18x1.45mm_HandSolder, F.Cu at (132.3, 78.2)
- added C4: C, Capacitor_SMD:C_Elec_5x5.8, F.Cu at (126.6, 86.8)
- added C5: C, Capacitor_SMD:C_0805_2012Metric_Pad1.18x1.45mm_HandSolder, F.Cu at (140.8, 99.8)
- added C6: C, Capacitor_SMD:C_Elec_5x5.8, F.Cu at (159.4, 80.0)
- added REF**: MountingHole_2.2mm_M2, MountingHole:MountingHole_2.2mm_M2, F.Cu at (159.7, 127.9)
- added U4: L7805, Package_TO_SOT_SMD:TO-263-3_TabPin2, F.Cu at (145.8, 73.2)
- moved J3 19.3 mm to (131.0, 67.9), turned to 90 degrees
- moved J4 18.4 mm to (126.5, 78.8)
- moved REF** 1.33 mm to (160.0, 68.2)
- moved REF** 1.32 mm to (125.8, 68.2)
- moved J1 0.91 mm to (143.6, 90.9), turned to 180 degrees
Routing:
- net SCL: track 23.9 -> 5.89 mm
- net SDA: track 19.6 -> 9.64 mm
- net +5V: track 71.8 -> 67.2 mm, vias 0 -> 1
- net +3V3: track 67.3 -> 63.1 mm, vias 1 -> 2
- net IO33: track 21.5 -> 17.6 mm
- net VCC: track 43.9 -> 46.7 mm, vias 0 -> 1
- net IO16: track 17.6 -> 16.3 mm
Other:
- board size 39.3 x 63.7 mm -> 39.3 x 65 mm
