File: Hardware/Swamper.kicad_sch (KiCad schematic)
At the start: 7 parts, among them J1 MPU6050, J2 Sensor de temperatura, J4 Entrada, U1 ESP32, U2 SEN-12650, U3 Mini360

Commit message: Actualizacion de repositorio
Parts:
- removed U3: Mini360, MixLib:Mini360_step-down, symbol MixLib:Mini360
- added C1, C4, C6: C, Capacitor_SMD:C_Elec_5x5.8, symbol Device:C
- added C2, C3, C5: C, Capacitor_SMD:C_0805_2012Metric_Pad1.18x1.45mm_HandSolder, symbol Device:C
- added U4: L7805, Package_TO_SOT_SMD:TO-263-3_TabPin2, symbol Regulator_Linear:L7805
Connections:
- net +3V3: now also C5.1, C6.1
- net +5V: now also C3.1, C4.1, U4.3 (OUT)
- net GND: now also C1.2, C2.2, C3.2, C4.2, C5.2, C6.2, U4.2 (GND)
- net VCC: now also C1.1, C2.1, U4.1 (IN)
Other:
- moved on the sheet: J1
